File: hardware/carrier32/carrier32.kicad_pcb (KiCad board)
At the start: 4 copper layers, 240 x 160 mm, 46 parts, among them J1 12V INPUT, Q1 AO4443, U3 AP2112K-3.3TRG1, U4 AP2112K-3.3TRG1

Commit message: feat: sync dual-node bench progress and Carrier32 draft
Parts:
- added C11: >=33u effective/16V X7R, Capacitor_SMD:C_1210_3225Metric, F.Cu at (215.0, 143.0)
- added C20: >=33u effective/16V X7R, Capacitor_SMD:C_1210_3225Metric, F.Cu at (221.0, 108.0)
- added C22: >=33u effective/16V X7R, Capacitor_SMD:C_1210_3225Metric, F.Cu at (221.0, 149.0)
- added C6: >=33u effective/16V X7R, Capacitor_SMD:C_1210_3225Metric, F.Cu at (215.0, 102.0)
- added D_WS01: WS2812-01, LED_SMD:LED_WS2812B_PLCC4_5.0x5.0mm_P3.2mm, F.Cu at (75.0, 274.0)
- added D_WS02: WS2812-02, LED_SMD:LED_WS2812B_PLCC4_5.0x5.0mm_P3.2mm, F.Cu at (109.0, 274.0)
- added D_WS03: WS2812-03, LED_SMD:LED_WS2812B_PLCC4_5.0x5.0mm_P3.2mm, F.Cu at (143.0, 274.0)
- added D_WS04: WS2812-04, LED_SMD:LED_WS2812B_PLCC4_5.0x5.0mm_P3.2mm, F.Cu at (177.0, 274.0)
- added D_WS05: WS2812-05, LED_SMD:LED_WS2812B_PLCC4_5.0x5.0mm_P3.2mm, F.Cu at (211.0, 274.0)
- added D_WS06: WS2812-06, LED_SMD:LED_WS2812B_PLCC4_5.0x5.0mm_P3.2mm, F.Cu at (245.0, 274.0)
- added D_WS07: WS2812-07, LED_SMD:LED_WS2812B_PLCC4_5.0x5.0mm_P3.2mm, F.Cu at (279.0, 274.0)
- added D_WS08: WS2812-08, LED_SMD:LED_WS2812B_PLCC4_5.0x5.0mm_P3.2mm, F.Cu at (313.0, 274.0)
- added D_WS09: WS2812-09, LED_SMD:LED_WS2812B_PLCC4_5.0x5.0mm_P3.2mm, F.Cu at (347.0, 274.0)
- added D_WS10: WS2812-10, LED_SMD:LED_WS2812B_PLCC4_5.0x5.0mm_P3.2mm, F.Cu at (75.0, 296.0)
- added D_WS11: WS2812-11, LED_SMD:LED_WS2812B_PLCC4_5.0x5.0mm_P3.2mm, F.Cu at (109.0, 296.0)
- added D_WS12: WS2812-12, LED_SMD:LED_WS2812B_PLCC4_5.0x5.0mm_P3.2mm, F.Cu at (143.0, 296.0)
- added D_WS13: WS2812-13, LED_SMD:LED_WS2812B_PLCC4_5.0x5.0mm_P3.2mm, F.Cu at (177.0, 296.0)
- added D_WS14: WS2812-14, LED_SMD:LED_WS2812B_PLCC4_5.0x5.0mm_P3.2mm, F.Cu at (211.0, 296.0)
- added D_WS15: WS2812-15, LED_SMD:LED_WS2812B_PLCC4_5.0x5.0mm_P3.2mm, F.Cu at (245.0, 296.0)
- added D_WS16: WS2812-16, LED_SMD:LED_WS2812B_PLCC4_5.0x5.0mm_P3.2mm, F.Cu at (279.0, 296.0)
- added D_WS17: WS2812-17, LED_SMD:LED_WS2812B_PLCC4_5.0x5.0mm_P3.2mm, F.Cu at (313.0, 296.0)
- added D_WS18: WS2812-18, LED_SMD:LED_WS2812B_PLCC4_5.0x5.0mm_P3.2mm, F.Cu at (347.0, 296.0)
- added F1: SELECT_BY_TEST, Fuse:Fuse_1210_3225Metric, F.Cu at (79.0, 60.0)
- added J_BUZZER: BUZZER, Connector_PinSocket_2.54mm:PinSocket_1x02_P2.54mm_Vertical, F.Cu at (395.0, 250.0)
- added J_ESP_A: ESP-01S-A, Connector_PinSocket_2.54mm:PinSocket_2x04_P2.54mm_Vertical, F.Cu at (320.0, 150.0)
- added J_ESP_B: ESP-01S-B, Connector_PinSocket_2.54mm:PinSocket_2x04_P2.54mm_Vertical, F.Cu at (375.0, 150.0)
- added J_FAN_A: FAN-A-12V-0.2A, Connector_JST:JST_XH_B4B-XH-A_1x04_P2.50mm_Vertical, F.Cu at (345.0, 220.0)
- added J_FAN_B: FAN-B-12V-0.2A, Connector_JST:JST_XH_B4B-XH-A_1x04_P2.50mm_Vertical, F.Cu at (375.0, 220.0)
- added J_FLAME01: FLAME-01, Connector_JST:JST_XH_B4B-XH-A_1x04_P2.50mm_Vertical, F.Cu at (68.0, 164.0)
- added J_FLAME02: FLAME-02, Connector_JST:JST_XH_B4B-XH-A_1x04_P2.50mm_Vertical, F.Cu at (96.0, 164.0)
- added J_FLAME03: FLAME-03, Connector_JST:JST_XH_B4B-XH-A_1x04_P2.50mm_Vertical, F.Cu at (124.0, 164.0)
- added J_FLAME04: FLAME-04, Connector_JST:JST_XH_B4B-XH-A_1x04_P2.50mm_Vertical, F.Cu at (152.0, 164.0)
- added J_FLAME05: FLAME-05, Connector_JST:JST_XH_B4B-XH-A_1x04_P2.50mm_Vertical, F.Cu at (180.0, 164.0)
- added J_INA_A: INA226-A, Connector_PinSocket_2.54mm:PinSocket_1x06_P2.54mm_Vertical, F.Cu at (315.0, 250.0)
- added J_INA_B: INA226-B, Connector_PinSocket_2.54mm:PinSocket_1x06_P2.54mm_Vertical, F.Cu at (345.0, 250.0)
- added J_JOY: JOYSTICK-B, Connector_PinSocket_2.54mm:PinSocket_1x05_P2.54mm_Vertical, F.Cu at (315.0, 220.0)
- added J_LEVEL01: LEVEL-01, Connector_JST:JST_XH_B4B-XH-A_1x04_P2.50mm_Vertical, F.Cu at (208.0, 164.0)
- added J_LEVEL02: LEVEL-02, Connector_JST:JST_XH_B4B-XH-A_1x04_P2.50mm_Vertical, F.Cu at (236.0, 164.0)
- added J_LEVEL03: LEVEL-03, Connector_JST:JST_XH_B4B-XH-A_1x04_P2.50mm_Vertical, F.Cu at (264.0, 164.0)
- added J_LEVEL04: LEVEL-04, Connector_JST:JST_XH_B4B-XH-A_1x04_P2.50mm_Vertical, F.Cu at (68.0, 177.0)
- added J_LEVEL05: LEVEL-05, Connector_JST:JST_XH_B4B-XH-A_1x04_P2.50mm_Vertical, F.Cu at (96.0, 177.0)
- added J_MCU_A: STM32F103RCT6-A, Connector_PinSocket_2.54mm:PinSocket_2x20_P2.54mm_Vertical, F.Cu at (320.0, 85.0)
- added J_MCU_B: STM32F103RCT6-B, Connector_PinSocket_2.54mm:PinSocket_2x20_P2.54mm_Vertical, F.Cu at (375.0, 85.0)
- added J_MQ201: MQ2-01, Connector_JST:JST_XH_B4B-XH-A_1x04_P2.50mm_Vertical, F.Cu at (124.0, 177.0)
- added J_MQ202: MQ2-02, Connector_JST:JST_XH_B4B-XH-A_1x04_P2.50mm_Vertical, F.Cu at (152.0, 177.0)
- added J_MQ203: MQ2-03, Connector_JST:JST_XH_B4B-XH-A_1x04_P2.50mm_Vertical, F.Cu at (180.0, 177.0)
- added J_MQ204: MQ2-04, Connector_JST:JST_XH_B4B-XH-A_1x04_P2.50mm_Vertical, F.Cu at (208.0, 177.0)
- added J_MQ205: MQ2-05, Connector_JST:JST_XH_B4B-XH-A_1x04_P2.50mm_Vertical, F.Cu at (236.0, 177.0)
- added J_MQ401: MQ4-01, Connector_JST:JST_XH_B4B-XH-A_1x04_P2.50mm_Vertical, F.Cu at (264.0, 177.0)
- added J_MQ402: MQ4-02, Connector_JST:JST_XH_B4B-XH-A_1x04_P2.50mm_Vertical, F.Cu at (68.0, 190.0)
- added J_MQ403: MQ4-03, Connector_JST:JST_XH_B4B-XH-A_1x04_P2.50mm_Vertical, F.Cu at (96.0, 190.0)
- added J_MQ404: MQ4-04, Connector_JST:JST_XH_B4B-XH-A_1x04_P2.50mm_Vertical, F.Cu at (124.0, 190.0)
- added J_MQ405: MQ4-05, Connector_JST:JST_XH_B4B-XH-A_1x04_P2.50mm_Vertical, F.Cu at (152.0, 190.0)
- added J_MQ701: MQ7-01, Connector_JST:JST_XH_B4B-XH-A_1x04_P2.50mm_Vertical, F.Cu at (180.0, 190.0)
- added J_MQ702: MQ7-02, Connector_JST:JST_XH_B4B-XH-A_1x04_P2.50mm_Vertical, F.Cu at (208.0, 190.0)
- added J_MQ703: MQ7-03, Connector_JST:JST_XH_B4B-XH-A_1x04_P2.50mm_Vertical, F.Cu at (236.0, 190.0)
- added J_MQ704: MQ7-04, Connector_JST:JST_XH_B4B-XH-A_1x04_P2.50mm_Vertical, F.Cu at (264.0, 190.0)
- added J_MQ705: MQ7-05, Connector_JST:JST_XH_B4B-XH-A_1x04_P2.50mm_Vertical, F.Cu at (68.0, 203.0)
- added J_O201: O2-01, Connector_JST:JST_XH_B4B-XH-A_1x04_P2.50mm_Vertical, F.Cu at (96.0, 203.0)
- added J_O202: O2-02, Connector_JST:JST_XH_B4B-XH-A_1x04_P2.50mm_Vertical, F.Cu at (124.0, 203.0)
- added J_O203: O2-03, Connector_JST:JST_XH_B4B-XH-A_1x04_P2.50mm_Vertical, F.Cu at (152.0, 203.0)
- added J_RELAY: RELAY, Connector_PinSocket_2.54mm:PinSocket_1x03_P2.54mm_Vertical, F.Cu at (375.0, 250.0)
- added J_SHT01: SHT-01, Connector_JST:JST_XH_B4B-XH-A_1x04_P2.50mm_Vertical, F.Cu at (180.0, 203.0)
- added J_SHT02: SHT-02, Connector_JST:JST_XH_B4B-XH-A_1x04_P2.50mm_Vertical, F.Cu at (208.0, 203.0)
- added J_SHT03: SHT-03, Connector_JST:JST_XH_B4B-XH-A_1x04_P2.50mm_Vertical, F.Cu at (236.0, 203.0)
- added J_SHT04: SHT-04, Connector_JST:JST_XH_B4B-XH-A_1x04_P2.50mm_Vertical, F.Cu at (264.0, 203.0)
- added J_TFT_A: ST7735S-A, Connector_PinSocket_2.54mm:PinSocket_1x08_P2.54mm_Vertical, F.Cu at (320.0, 185.0)
- added J_TFT_B: ST7735S-B, Connector_PinSocket_2.54mm:PinSocket_1x08_P2.54mm_Vertical, F.Cu at (375.0, 185.0)
- added L1: 4.7uH >=6A RMS, >=10A ISAT, Inductor_SMD:L_Abracon_ASPI-0628, F.Cu at (181.0, 95.0)
- added L2: 4.7uH >=6A RMS, >=10A ISAT, Inductor_SMD:L_Abracon_ASPI-0628, F.Cu at (181.0, 133.0)
- added U1: LMR51450FSQDRRRQ1 (LOGIC), Carrier32:LMR51450_visual_13pin, F.Cu at (220.0, 77.0)
- added U2: LMR51450FSQDRRRQ1 (MQ), Carrier32:LMR51450_visual_13pin, F.Cu at (220.0, 124.0)
- F10, F2, F3, F4, F5, F6, F7, F8, F9: footprint Fuse:Fuse_1812_4532Metric -> Fuse:Fuse_1210_3225Metric
Other:
- board size 240 x 160 mm -> 360 x 260 mm
- board text added: "CARRIER32 VISUAL DEMO"
- board text added: "MCU AND MODULES"
- board text added: "POWER DISTRIBUTION"
- board text added: "SENSOR PORTS 32"
- board text added: "WS2812 RGB 18"
