File: hardware/carrier32/carrier32.kicad_sch (KiCad schematic)
At the start: 55 parts, among them J1 12V INPUT, Q1 AO4443, U1 LMR51450FSQDRRRQ1 (LOGIC), U2 LMR51450FSQDRRRQ1 (MQ), U3 AP2112K-3.3TRG1, U4 AP2112K-3.3TRG1

Commit message: feat: sync dual-node bench progress and Carrier32 draft
Parts:
- added D_WS01: WS2812-01, LED_SMD:LED_WS2812B_PLCC4_5.0x5.0mm_P3.2mm, symbol LED:WS2812B
- added D_WS02: WS2812-02, LED_SMD:LED_WS2812B_PLCC4_5.0x5.0mm_P3.2mm, symbol LED:WS2812B
- added D_WS03: WS2812-03, LED_SMD:LED_WS2812B_PLCC4_5.0x5.0mm_P3.2mm, symbol LED:WS2812B
- added D_WS04: WS2812-04, LED_SMD:LED_WS2812B_PLCC4_5.0x5.0mm_P3.2mm, symbol LED:WS2812B
- added D_WS05: WS2812-05, LED_SMD:LED_WS2812B_PLCC4_5.0x5.0mm_P3.2mm, symbol LED:WS2812B
- added D_WS06: WS2812-06, LED_SMD:LED_WS2812B_PLCC4_5.0x5.0mm_P3.2mm, symbol LED:WS2812B
- added D_WS07: WS2812-07, LED_SMD:LED_WS2812B_PLCC4_5.0x5.0mm_P3.2mm, symbol LED:WS2812B
- added D_WS08: WS2812-08, LED_SMD:LED_WS2812B_PLCC4_5.0x5.0mm_P3.2mm, symbol LED:WS2812B
- added D_WS09: WS2812-09, LED_SMD:LED_WS2812B_PLCC4_5.0x5.0mm_P3.2mm, symbol LED:WS2812B
- added D_WS10: WS2812-10, LED_SMD:LED_WS2812B_PLCC4_5.0x5.0mm_P3.2mm, symbol LED:WS2812B
- added D_WS11: WS2812-11, LED_SMD:LED_WS2812B_PLCC4_5.0x5.0mm_P3.2mm, symbol LED:WS2812B
- added D_WS12: WS2812-12, LED_SMD:LED_WS2812B_PLCC4_5.0x5.0mm_P3.2mm, symbol LED:WS2812B
- added D_WS13: WS2812-13, LED_SMD:LED_WS2812B_PLCC4_5.0x5.0mm_P3.2mm, symbol LED:WS2812B
- added D_WS14: WS2812-14, LED_SMD:LED_WS2812B_PLCC4_5.0x5.0mm_P3.2mm, symbol LED:WS2812B
- added D_WS15: WS2812-15, LED_SMD:LED_WS2812B_PLCC4_5.0x5.0mm_P3.2mm, symbol LED:WS2812B
- added D_WS16: WS2812-16, LED_SMD:LED_WS2812B_PLCC4_5.0x5.0mm_P3.2mm, symbol LED:WS2812B
- added D_WS17: WS2812-17, LED_SMD:LED_WS2812B_PLCC4_5.0x5.0mm_P3.2mm, symbol LED:WS2812B
- added D_WS18: WS2812-18, LED_SMD:LED_WS2812B_PLCC4_5.0x5.0mm_P3.2mm, symbol LED:WS2812B
- added J_BUZZER: BUZZER, Connector_PinSocket_2.54mm:PinSocket_1x02_P2.54mm_Vertical, symbol Connector_Generic:Conn_01x02
- added J_ESP_A: ESP-01S-A, Connector_PinSocket_2.54mm:PinSocket_2x04_P2.54mm_Vertical, symbol Connector_Generic:Conn_02x04_Odd_Even
- added J_ESP_B: ESP-01S-B, Connector_PinSocket_2.54mm:PinSocket_2x04_P2.54mm_Vertical, symbol Connector_Generic:Conn_02x04_Odd_Even
- added J_FAN_A: FAN-A-12V-0.2A, Connector_JST:JST_XH_B4B-XH-A_1x04_P2.50mm_Vertical, symbol Connector_Generic:Conn_01x04
- added J_FAN_B: FAN-B-12V-0.2A, Connector_JST:JST_XH_B4B-XH-A_1x04_P2.50mm_Vertical, symbol Connector_Generic:Conn_01x04
- added J_FLAME01: FLAME-01, Connector_JST:JST_XH_B4B-XH-A_1x04_P2.50mm_Vertical, symbol Connector_Generic:Conn_01x04
- added J_FLAME02: FLAME-02, Connector_JST:JST_XH_B4B-XH-A_1x04_P2.50mm_Vertical, symbol Connector_Generic:Conn_01x04
- added J_FLAME03: FLAME-03, Connector_JST:JST_XH_B4B-XH-A_1x04_P2.50mm_Vertical, symbol Connector_Generic:Conn_01x04
- added J_FLAME04: FLAME-04, Connector_JST:JST_XH_B4B-XH-A_1x04_P2.50mm_Vertical, symbol Connector_Generic:Conn_01x04
- added J_FLAME05: FLAME-05, Connector_JST:JST_XH_B4B-XH-A_1x04_P2.50mm_Vertical, symbol Connector_Generic:Conn_01x04
- added J_INA_A: INA226-A, Connector_PinSocket_2.54mm:PinSocket_1x06_P2.54mm_Vertical, symbol Connector_Generic:Conn_01x06
- added J_INA_B: INA226-B, Connector_PinSocket_2.54mm:PinSocket_1x06_P2.54mm_Vertical, symbol Connector_Generic:Conn_01x06
- added J_JOY: JOYSTICK-B, Connector_PinSocket_2.54mm:PinSocket_1x05_P2.54mm_Vertical, symbol Connector_Generic:Conn_01x05
- added J_LEVEL01: LEVEL-01, Connector_JST:JST_XH_B4B-XH-A_1x04_P2.50mm_Vertical, symbol Connector_Generic:Conn_01x04
- added J_LEVEL02: LEVEL-02, Connector_JST:JST_XH_B4B-XH-A_1x04_P2.50mm_Vertical, symbol Connector_Generic:Conn_01x04
- added J_LEVEL03: LEVEL-03, Connector_JST:JST_XH_B4B-XH-A_1x04_P2.50mm_Vertical, symbol Connector_Generic:Conn_01x04
- added J_LEVEL04: LEVEL-04, Connector_JST:JST_XH_B4B-XH-A_1x04_P2.50mm_Vertical, symbol Connector_Generic:Conn_01x04
- added J_LEVEL05: LEVEL-05, Connector_JST:JST_XH_B4B-XH-A_1x04_P2.50mm_Vertical, symbol Connector_Generic:Conn_01x04
- added J_MCU_A: STM32F103RCT6-A, Connector_PinSocket_2.54mm:PinSocket_2x20_P2.54mm_Vertical, symbol Connector_Generic:Conn_02x20_Odd_Even
- added J_MCU_B: STM32F103RCT6-B, Connector_PinSocket_2.54mm:PinSocket_2x20_P2.54mm_Vertical, symbol Connector_Generic:Conn_02x20_Odd_Even
- added J_MQ201: MQ2-01, Connector_JST:JST_XH_B4B-XH-A_1x04_P2.50mm_Vertical, symbol Connector_Generic:Conn_01x04
- added J_MQ202: MQ2-02, Connector_JST:JST_XH_B4B-XH-A_1x04_P2.50mm_Vertical, symbol Connector_Generic:Conn_01x04
- added J_MQ203: MQ2-03, Connector_JST:JST_XH_B4B-XH-A_1x04_P2.50mm_Vertical, symbol Connector_Generic:Conn_01x04
- added J_MQ204: MQ2-04, Connector_JST:JST_XH_B4B-XH-A_1x04_P2.50mm_Vertical, symbol Connector_Generic:Conn_01x04
- added J_MQ205: MQ2-05, Connector_JST:JST_XH_B4B-XH-A_1x04_P2.50mm_Vertical, symbol Connector_Generic:Conn_01x04
- added J_MQ401: MQ4-01, Connector_JST:JST_XH_B4B-XH-A_1x04_P2.50mm_Vertical, symbol Connector_Generic:Conn_01x04
- added J_MQ402: MQ4-02, Connector_JST:JST_XH_B4B-XH-A_1x04_P2.50mm_Vertical, symbol Connector_Generic:Conn_01x04
- added J_MQ403: MQ4-03, Connector_JST:JST_XH_B4B-XH-A_1x04_P2.50mm_Vertical, symbol Connector_Generic:Conn_01x04
- added J_MQ404: MQ4-04, Connector_JST:JST_XH_B4B-XH-A_1x04_P2.50mm_Vertical, symbol Connector_Generic:Conn_01x04
- added J_MQ405: MQ4-05, Connector_JST:JST_XH_B4B-XH-A_1x04_P2.50mm_Vertical, symbol Connector_Generic:Conn_01x04
- added J_MQ701: MQ7-01, Connector_JST:JST_XH_B4B-XH-A_1x04_P2.50mm_Vertical, symbol Connector_Generic:Conn_01x04
- added J_MQ702: MQ7-02, Connector_JST:JST_XH_B4B-XH-A_1x04_P2.50mm_Vertical, symbol Connector_Generic:Conn_01x04
- added J_MQ703: MQ7-03, Connector_JST:JST_XH_B4B-XH-A_1x04_P2.50mm_Vertical, symbol Connector_Generic:Conn_01x04
- added J_MQ704: MQ7-04, Connector_JST:JST_XH_B4B-XH-A_1x04_P2.50mm_Vertical, symbol Connector_Generic:Conn_01x04
- added J_MQ705: MQ7-05, Connector_JST:JST_XH_B4B-XH-A_1x04_P2.50mm_Vertical, symbol Connector_Generic:Conn_01x04
- added J_O201: O2-01, Connector_JST:JST_XH_B4B-XH-A_1x04_P2.50mm_Vertical, symbol Connector_Generic:Conn_01x04
- added J_O202: O2-02, Connector_JST:JST_XH_B4B-XH-A_1x04_P2.50mm_Vertical, symbol Connector_Generic:Conn_01x04
- added J_O203: O2-03, Connector_JST:JST_XH_B4B-XH-A_1x04_P2.50mm_Vertical, symbol Connector_Generic:Conn_01x04
- added J_RELAY: RELAY, Connector_PinSocket_2.54mm:PinSocket_1x03_P2.54mm_Vertical, symbol Connector_Generic:Conn_01x03
- added J_SHT01: SHT-01, Connector_JST:JST_XH_B4B-XH-A_1x04_P2.50mm_Vertical, symbol Connector_Generic:Conn_01x04
- added J_SHT02: SHT-02, Connector_JST:JST_XH_B4B-XH-A_1x04_P2.50mm_Vertical, symbol Connector_Generic:Conn_01x04
- added J_SHT03: SHT-03, Connector_JST:JST_XH_B4B-XH-A_1x04_P2.50mm_Vertical, symbol Connector_Generic:Conn_01x04
- added J_SHT04: SHT-04, Connector_JST:JST_XH_B4B-XH-A_1x04_P2.50mm_Vertical, symbol Connector_Generic:Conn_01x04
- added J_TFT_A: ST7735S-A, Connector_PinSocket_2.54mm:PinSocket_1x08_P2.54mm_Vertical, symbol Connector_Generic:Conn_01x08
- added J_TFT_B: ST7735S-B, Connector_PinSocket_2.54mm:PinSocket_1x08_P2.54mm_Vertical, symbol Connector_Generic:Conn_01x08
- C11, C20, C22, C6: footprint (none) -> Capacitor_SMD:C_1210_3225Metric
- F1: footprint (none) -> Fuse:Fuse_1210_3225Metric
- F10, F2, F3, F4, F5, F6, F7, F8, F9: footprint Fuse:Fuse_1812_4532Metric -> Fuse:Fuse_1210_3225Metric
- L1, L2: footprint (none) -> Inductor_SMD:L_Abracon_ASPI-0628
- U1, U2: footprint (none) -> Carrier32:LMR51450_visual_13pin
Connections:
- net 12V_FAN_A: now also J_FAN_A.2 (Pin_2), J_INA_A.6 (Pin_6)
- net 12V_FAN_B: now also J_FAN_B.2 (Pin_2), J_INA_B.6 (Pin_6)
- net 12V_PROTECTED: now also J_INA_A.5 (Pin_5), J_INA_B.5 (Pin_5)
- net 3V3_ESP_A: now also J_ESP_A.2 (Pin_2), J_ESP_A.5 (Pin_5), J_ESP_A.6 (Pin_6), J_ESP_A.7 (Pin_7), J_ESP_A.8 (Pin_8)
- net 3V3_ESP_B: now also J_ESP_B.2 (Pin_2), J_ESP_B.5 (Pin_5), J_ESP_B.6 (Pin_6), J_ESP_B.7 (Pin_7), J_ESP_B.8 (Pin_8)
- net 5V_LOGIC: now also J_MCU_A.22 (Pin_22), J_MCU_B.14 (Pin_14)
- net 5V_MQ2: now also J_MQ201.2 (Pin_2), J_MQ202.2 (Pin_2), J_MQ203.2 (Pin_2), J_MQ204.2 (Pin_2), J_MQ205.2 (Pin_2)
- net 5V_MQ4: now also J_MQ401.2 (Pin_2), J_MQ402.2 (Pin_2), J_MQ403.2 (Pin_2), J_MQ404.2 (Pin_2), J_MQ405.2 (Pin_2)
- net 5V_MQ7: now also J_MQ701.2 (Pin_2), J_MQ702.2 (Pin_2), J_MQ703.2 (Pin_2), J_MQ704.2 (Pin_2), J_MQ705.2 (Pin_2)
- net 5V_RELAY: now also J_RELAY.2 (Pin_2)
- net 5V_SENSORS: now also J_FLAME01.2 (Pin_2), J_FLAME02.2 (Pin_2), J_FLAME03.2 (Pin_2), J_FLAME04.2 (Pin_2), J_FLAME05.2 (Pin_2), J_LEVEL01.2 (Pin_2), J_LEVEL02.2 (Pin_2), J_LEVEL03.2 (Pin_2), J_LEVEL04.2 (Pin_2), J_LEVEL05.2 (Pin_2), J_O201.2 (Pin_2), J_O202.2 (Pin_2), J_O203.2 (Pin_2)
- net 5V_WS: now also D_WS01.1 (VDD), D_WS02.1 (VDD), D_WS03.1 (VDD), D_WS04.1 (VDD), D_WS05.1 (VDD), D_WS06.1 (VDD), D_WS07.1 (VDD), D_WS08.1 (VDD), D_WS09.1 (VDD), D_WS10.1 (VDD), D_WS11.1 (VDD), D_WS12.1 (VDD), D_WS13.1 (VDD), D_WS14.1 (VDD), D_WS15.1 (VDD), D_WS16.1 (VDD), D_WS17.1 (VDD), D_WS18.1 (VDD)
- net GND: now also D_WS01.3 (VSS), D_WS02.3 (VSS), D_WS03.3 (VSS), D_WS04.3 (VSS), D_WS05.3 (VSS), D_WS06.3 (VSS), D_WS07.3 (VSS), D_WS08.3 (VSS), D_WS09.3 (VSS), D_WS10.3 (VSS), D_WS11.3 (VSS), D_WS12.3 (VSS), D_WS13.3 (VSS), D_WS14.3 (VSS), D_WS15.3 (VSS), D_WS16.3 (VSS), D_WS17.3 (VSS), D_WS18.3 (VSS), J_BUZZER.1 (Pin_1), J_ESP_A.1 (Pin_1), J_ESP_B.1 (Pin_1), J_FAN_A.1 (Pin_1), J_FAN_B.1 (Pin_1), J_FLAME01.1 (Pin_1), J_FLAME02.1 (Pin_1), J_FLAME03.1 (Pin_1), J_FLAME04.1 (Pin_1), J_FLAME05.1 (Pin_1), J_INA_A.1 (Pin_1), J_INA_B.1 (Pin_1), J_JOY.1 (Pin_1), J_LEVEL01.1 (Pin_1), J_LEVEL02.1 (Pin_1), J_LEVEL03.1 (Pin_1), J_LEVEL04.1 (Pin_1), J_LEVEL05.1 (Pin_1), J_MCU_A.21 (Pin_21), J_MCU_B.13 (Pin_13), J_MQ201.1 (Pin_1), J_MQ202.1 (Pin_1), J_MQ203.1 (Pin_1), J_MQ204.1 (Pin_1), J_MQ205.1 (Pin_1), J_MQ401.1 (Pin_1), J_MQ402.1 (Pin_1), J_MQ403.1 (Pin_1), J_MQ404.1 (Pin_1), J_MQ405.1 (Pin_1), J_MQ701.1 (Pin_1), J_MQ702.1 (Pin_1), J_MQ703.1 (Pin_1), J_MQ704.1 (Pin_1), J_MQ705.1 (Pin_1), J_O201.1 (Pin_1), J_O202.1 (Pin_1), J_O203.1 (Pin_1), J_RELAY.1 (Pin_1), J_SHT01.1 (Pin_1), J_SHT02.1 (Pin_1), J_SHT03.1 (Pin_1), J_SHT04.1 (Pin_1), J_TFT_A.1 (Pin_1), J_TFT_B.1 (Pin_1)
- new net 3V3_SENSORS: J_INA_A.2 (Pin_2), J_INA_B.2 (Pin_2), J_JOY.2 (Pin_2), J_MCU_A.23 (Pin_23), J_MCU_B.15 (Pin_15), J_SHT01.2 (Pin_2), J_SHT02.2 (Pin_2), J_SHT03.2 (Pin_2), J_SHT04.2 (Pin_2), J_TFT_A.2 (Pin_2), J_TFT_A.8 (Pin_8), J_TFT_B.2 (Pin_2), J_TFT_B.8 (Pin_8)
- new net A_BUZZ_CTRL: J_BUZZER.2 (Pin_2), J_MCU_A.40 (Pin_40)
- new net A_ESP_RX: J_ESP_A.4 (Pin_4), J_MCU_A.25 (Pin_25)
- new net A_ESP_TX: J_ESP_A.3 (Pin_3), J_MCU_A.24 (Pin_24)
- new net A_FAN_PWM: J_FAN_A.4 (Pin_4), J_MCU_A.35 (Pin_35)
- new net A_FAN_TACH: J_FAN_A.3 (Pin_3), J_MCU_A.36 (Pin_36)
- new net A_INA_SCL: J_INA_A.3 (Pin_3), J_MCU_A.37 (Pin_37)
- new net A_INA_SDA: J_INA_A.4 (Pin_4), J_MCU_A.38 (Pin_38)
- new net A_JOY_SW: J_JOY.5 (Pin_5), J_MCU_A.33 (Pin_33)
- new net A_JOY_X: J_JOY.3 (Pin_3), J_MCU_A.31 (Pin_31)
- new net A_JOY_Y: J_JOY.4 (Pin_4), J_MCU_A.32 (Pin_32)
- new net A_PA0: J_MCU_A.1 (Pin_1), J_MQ702.3 (Pin_3)
- new net A_PA4: J_MCU_A.2 (Pin_2), J_MQ402.3 (Pin_3)
- new net A_PA5: J_MCU_A.3 (Pin_3), J_O202.3 (Pin_3)
- new net A_PB1: J_MCU_A.4 (Pin_4), J_MQ703.3 (Pin_3)
- new net A_PB10_SCL: J_MCU_A.5 (Pin_5), J_SHT03.4 (Pin_4), J_SHT04.4 (Pin_4)
- new net A_PB11_SDA: J_MCU_A.6 (Pin_6), J_SHT03.3 (Pin_3), J_SHT04.3 (Pin_3)
- new net A_PB12: J_MCU_A.7 (Pin_7), J_MQ201.3 (Pin_3)
- new net A_PB14: J_FLAME01.3 (Pin_3), J_MCU_A.8 (Pin_8)
- new net A_PB6_SCL: J_MCU_A.9 (Pin_9), J_SHT01.4 (Pin_4), J_SHT02.4 (Pin_4)
- new net A_PB7_SDA: J_MCU_A.10 (Pin_10), J_SHT01.3 (Pin_3), J_SHT02.3 (Pin_3)
- new net A_PC0: J_LEVEL01.3 (Pin_3), J_MCU_A.11 (Pin_11)
- new net A_PC1: J_MCU_A.12 (Pin_12), J_MQ701.3 (Pin_3)
- new net A_PC10: J_MCU_A.13 (Pin_13), J_MQ202.3 (Pin_3)
- new net A_PC11: J_MCU_A.14 (Pin_14), J_MQ203.3 (Pin_3)
- new net A_PC12: J_LEVEL02.3 (Pin_3), J_MCU_A.15 (Pin_15)
- new net A_PC13: J_LEVEL03.3 (Pin_3), J_MCU_A.16 (Pin_16)
- new net A_PC2: J_MCU_A.17 (Pin_17), J_MQ401.3 (Pin_3)
- new net A_PC3: J_MCU_A.18 (Pin_18), J_O201.3 (Pin_3)
- new net A_PC8: J_FLAME02.3 (Pin_3), J_MCU_A.19 (Pin_19)
- new net A_PC9: J_FLAME03.3 (Pin_3), J_MCU_A.20 (Pin_20)
- new net A_RELAY_CTRL: J_MCU_A.39 (Pin_39), J_RELAY.3 (Pin_3)
- new net A_TFT_CS: J_MCU_A.28 (Pin_28), J_TFT_A.5 (Pin_5)
- new net A_TFT_DC: J_MCU_A.29 (Pin_29), J_TFT_A.6 (Pin_6)
- new net A_TFT_MOSI: J_MCU_A.27 (Pin_27), J_TFT_A.4 (Pin_4)
- new net A_TFT_RST: J_MCU_A.30 (Pin_30), J_TFT_A.7 (Pin_7)
- new net A_TFT_SCK: J_MCU_A.26 (Pin_26), J_TFT_A.3 (Pin_3)
- new net A_WS_DATA: D_WS01.4 (DIN), J_MCU_A.34 (Pin_34)
- new net B_ESP_RX: J_ESP_B.4 (Pin_4), J_MCU_B.17 (Pin_17)
- new net B_ESP_TX: J_ESP_B.3 (Pin_3), J_MCU_B.16 (Pin_16)
- new net B_FAN_PWM: J_FAN_B.4 (Pin_4), J_MCU_B.24 (Pin_24)
- new net B_FAN_TACH: J_FAN_B.3 (Pin_3), J_MCU_B.25 (Pin_25)
- new net B_INA_SCL: J_INA_B.3 (Pin_3), J_MCU_B.26 (Pin_26)
- new net B_INA_SDA: J_INA_B.4 (Pin_4), J_MCU_B.27 (Pin_27)
- new net B_PA0: J_MCU_B.1 (Pin_1), J_MQ403.3 (Pin_3)
- new net B_PA1: J_MCU_B.2 (Pin_2), J_MQ404.3 (Pin_3)
- new net B_PA4: J_MCU_B.3 (Pin_3), J_MQ405.3 (Pin_3)
- new net B_PA6: J_MCU_B.4 (Pin_4), J_O203.3 (Pin_3)
- new net B_PB0: J_MCU_B.5 (Pin_5), J_MQ704.3 (Pin_3)
- new net B_PB1: J_MCU_B.6 (Pin_6), J_MQ705.3 (Pin_3)
- new net B_PC10: J_LEVEL04.3 (Pin_3), J_MCU_B.7 (Pin_7)
- new net B_PC11: J_LEVEL05.3 (Pin_3), J_MCU_B.8 (Pin_8)
- new net B_PC6: J_FLAME04.3 (Pin_3), J_MCU_B.9 (Pin_9)
- new net B_PC7: J_FLAME05.3 (Pin_3), J_MCU_B.10 (Pin_10)
- new net B_PC8: J_MCU_B.11 (Pin_11), J_MQ204.3 (Pin_3)
- new net B_PC9: J_MCU_B.12 (Pin_12), J_MQ205.3 (Pin_3)
- new net B_TFT_CS: J_MCU_B.20 (Pin_20), J_TFT_B.5 (Pin_5)
- new net B_TFT_DC: J_MCU_B.21 (Pin_21), J_TFT_B.6 (Pin_6)
- new net B_TFT_MOSI: J_MCU_B.19 (Pin_19), J_TFT_B.4 (Pin_4)
- new net B_TFT_RST: J_MCU_B.22 (Pin_22), J_TFT_B.7 (Pin_7)
- new net B_TFT_SCK: J_MCU_B.18 (Pin_18), J_TFT_B.3 (Pin_3)
- new net B_WS_DATA: D_WS10.4 (DIN), J_MCU_B.23 (Pin_23)
- new net WS_LINK_01: D_WS01.2 (DOUT), D_WS02.4 (DIN)
- new net WS_LINK_02: D_WS02.2 (DOUT), D_WS03.4 (DIN)
- new net WS_LINK_03: D_WS03.2 (DOUT), D_WS04.4 (DIN)
- new net WS_LINK_04: D_WS04.2 (DOUT), D_WS05.4 (DIN)
- new net WS_LINK_05: D_WS05.2 (DOUT), D_WS06.4 (DIN)
- new net WS_LINK_06: D_WS06.2 (DOUT), D_WS07.4 (DIN)
- new net WS_LINK_07: D_WS07.2 (DOUT), D_WS08.4 (DIN)
- new net WS_LINK_08: D_WS08.2 (DOUT), D_WS09.4 (DIN)
- new net WS_LINK_10: D_WS10.2 (DOUT), D_WS11.4 (DIN)
- new net WS_LINK_11: D_WS11.2 (DOUT), D_WS12.4 (DIN)
- new net WS_LINK_12: D_WS12.2 (DOUT), D_WS13.4 (DIN)
- new net WS_LINK_13: D_WS13.2 (DOUT), D_WS14.4 (DIN)
- new net WS_LINK_14: D_WS14.2 (DOUT), D_WS15.4 (DIN)
- new net WS_LINK_15: D_WS15.2 (DOUT), D_WS16.4 (DIN)
- new net WS_LINK_16: D_WS16.2 (DOUT), D_WS17.4 (DIN)
- new net WS_LINK_17: D_WS17.2 (DOUT), D_WS18.4 (DIN)
- no-connect marks 0 -> 43
Other:
- title: API Series 500 (EDA 306) -> Carrier32 visual demo schematic
